File: schematics/nav6.brd (EAGLE design)
At the start: 48.3 x 63.5 mm, 60 parts, among them J1 AVR_SPI_PRG_6PTH, Q1 MOSFET-N, Q2 MOSFET-N, U1 MAX232TSSOP, U2 ATMEGA168, X2 RS-232, Y1 16MHz

Commit message: Fixed up the headers in the file to reflect correct licensing information and attribution.
Parts:
- added U$1: CREATIVE_COMMONS, SparkFun:CREATIVE_COMMONS
Changed lines of the file:
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@@
 <element name="C1" library="SparkFun" package="0805" value="0.1uF" x="63.5" y="43.18" rot="R180"/>
 <element name="C2" library="SparkFun" package="0805" value="0.1uF" x="48.26" y="43.18" rot="R90"/>
+<element name="U$1" library="SparkFun" package="CREATIVE_COMMONS" value="CREATIVE_COMMONS" x="39.37" y="-7.62"/>
 </elements>
 <signals>
