File: schematics/nav6.sch (EAGLE design)
At the start: 56 parts, among them J1 AVR_SPI_PRG_6PTH, Q1 MOSFET-N, Q2 MOSFET-N, U1 MAX232TSSOP, U2 ATMEGA168, X2 RS-232, Y1 16MHz

Commit message: Fixed up the headers in the file to reflect correct licensing information and attribution.
Parts:
- added U$1: CREATIVE_COMMONS, SparkFun:CREATIVE_COMMONS
Other:
- note added: "KauaiLabs.com"
- note added: "Portions of this work are based on theopen-source ArduIMU project."
- note added: "Scott Libert, 2013"
Changed lines of the file:
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@@
 <part name="GND4" library="SparkFun" deviceset="GND" device=""/>
 <part name="P+1" library="SparkFun" deviceset="5V" device=""/>
+<part name="U$1" library="SparkFun" deviceset="CREATIVE_COMMONS" device=""/>
 </parts>
 <sheets>
@@
 <text x="275.59" y="63.5" size="4.064" layer="95">COMPASS</text>
 <text x="266.7" y="7.62" size="1.778" layer="91">I2C Address:  x1E (x3C Write, x3D Read)</text>
+<text x="53.34" y="203.2" size="5.08" layer="95">KauaiLabs.com</text>
+<text x="70.104" y="193.04" size="1.778" layer="95">Scott Libert, 2013</text>
+<text x="53.34" y="189.992" size="1.778" layer="95">Portions of this work are based on theopen-source ArduIMU project.</text>
 </plain>
 <instances>
@@
 <instance part="GND4" gate="1" x="154.94" y="50.8"/>
 <instance part="P+1" gate="G$1" x="43.18" y="152.4"/>
+<instance part="U$1" gate="G$1" x="53.34" y="193.04"/>
 </instances>
 <busses>
